Commit message: Multirobot support

File: bebop_description/urdf/bebop_base.urdf.xacro (robot description, xacro)
@@ -5,9 +5,10 @@
   <xacro:property name="camera_offset_len" value="0.1" />
   <xacro:property name="camera_offset_ver" value="0.0" />
-  <!-- +- 35 degrees -->
+  <!-- -35 .. +35 degrees -->
   <xacro:property name="pan_range" value="0.6108652381980153" />
   <xacro:property name="pan_vel" value="2.0" />
-  <!-- +- 35 degrees -->
-  <xacro:property name="tilt_range" value="0.6108652381980153" />
+  <!-- -90 .. +17 degrees -->
+  <xacro:property name="max_tilt" value="0.6108652381980153" />
+  <xacro:property name="min_tilt" value="-1.570796327" />
   <xacro:property name="tilt_vel" value="2.0" />
   <xacro:property name="joint_effort" value="50" />
@@ -35,5 +36,5 @@
     <child link="camera_tilt_link" />
     <axis xyz="0 1 0" />
-    <limit lower="${-tilt_range}" upper="${tilt_range}"
+    <limit lower="${min_tilt}" upper="${max_tilt}"
       effort="${joint_effort}" velocity="${tilt_vel}" />
   </joint>

Commit message: Added simple visual model to urdf description

File: bebop_description/urdf/bebop_base.urdf.xacro (robot description, xacro)
@@ -1,4 +1,4 @@
 <?xml version="1.0"?>
-<!-- Kinematic model only, no visuals, no collisions -->
+<!-- Kinematic model, simplified visual, no collisions -->
 <robot name="bebop" xmlns:xacro="http://www.ros.org/wiki/xacro">
   <xacro:property name="PI" value="3.1415926535897931" />
@@ -12,5 +12,11 @@
   <xacro:property name="tilt_vel" value="2.0" />
   <xacro:property name="joint_effort" value="50" />
-  <link name="base_link"></link>
+  <link name="base_link">
+   <visual>
+      <geometry>
+        <mesh scale=".001 .001 .001" filename="package://bebop_description/meshes/bebop_model.stl"/>
+      </geometry>
+   </visual>
+  </link>
   <link name="camera_base_link"></link>
   <link name="camera_pan_link"></link>

Commit message: Added mesh file from a different branch of bebop_autonomy. Fixed orientation of the model. Need to adjust the offset of mesh to be in line with the base frame. Need to verify optical frame offset from base frame.

File: bebop_description/urdf/bebop_base.urdf.xacro (robot description, xacro)
@@ -1,4 +1,4 @@
 <?xml version="1.0"?>
-<!-- Kinematic model only, no visuals, no collisions -->
+<!-- Kinematic model, simplified visual, no collisions -->
 <robot name="bebop" xmlns:xacro="http://www.ros.org/wiki/xacro">
   <xacro:property name="PI" value="3.1415926535897931" />
@@ -12,5 +12,12 @@
   <xacro:property name="tilt_vel" value="2.0" />
   <xacro:property name="joint_effort" value="50" />
-  <link name="base_link"></link>
+  <link name="base_link">
+   <visual>
+    	  <origin rpy="0 -0.0254 0" xyz="0 0 0"/>
+      <geometry>
+        <mesh filename="package://bebop_description/meshes/bebop_model.stl"/>
+      </geometry>
+   </visual>
+  </link>
   <link name="camera_base_link"></link>
   <link name="camera_pan_link"></link>

Commit message: Fixed URDF mesh offsets as well as camera frame offsets.

File: bebop_description/urdf/bebop_base.urdf.xacro (robot description, xacro)
@@ -3,5 +3,5 @@
 <robot name="bebop" xmlns:xacro="http://www.ros.org/wiki/xacro">
   <xacro:property name="PI" value="3.1415926535897931" />
-  <xacro:property name="camera_offset_len" value="0.1" />
+  <xacro:property name="camera_offset_len" value="0.1651" />
   <xacro:property name="camera_offset_ver" value="0.0" />
   <!-- +- 35 degrees -->
@@ -14,5 +14,5 @@
   <link name="base_link">
    <visual>
-    	  <origin rpy="0 -0.0254 0" xyz="0 0 0"/>
+    	  <origin xyz="0 -.0225 -0.02" rpy="0 -0.0254 0"/>
       <geometry>
         <mesh filename="package://bebop_description/meshes/bebop_model.stl"/>

Commit message: Fixed model size

File: bebop_description/urdf/bebop_base.urdf.xacro (robot description, xacro)
@@ -15,5 +15,5 @@
    <visual>
       <geometry>
-        <mesh scale=".001 .001 .001" filename="package://bebop_description/meshes/bebop_model.stl"/>
+        <mesh scale="1.0 1.0 1.0" filename="package://bebop_description/meshes/bebop_model.stl"/>
       </geometry>
    </visual>

Commit message: Removed model vertices for optimization, and improved the colour a bit.

File: bebop_description/urdf/bebop_base.urdf.xacro (robot description, xacro)
@@ -17,4 +17,7 @@
         <mesh scale="1.0 1.0 1.0" filename="package://bebop_description/meshes/bebop_model.stl"/>
       </geometry>
+        <material name="blue">
+          <color rgba="0 0.4 0.6 1"/>
+        </material>
    </visual>
   </link>
